File: stm_audio_board_v3_Footswitch/stm_audio_board_v3_Footswitch.kicad_pcb (KiCad board)
At the start: 2 copper layers, 9 parts, among them J2 Conn_01x10_Footswitch, SW1 3PDT, SW2 3PDT, SW3 3PDT, SW4 3PDT

Commit message: Problem with new footprint grid and pin assignements
Connections:
- D1 pad 1: unconnected-(D1-K-Pad1) -> GND
- D1 pad 2: unconnected-(D1-A-Pad2) -> LED1
- D2 pad 1: unconnected-(D2-K-Pad1) -> GND
- D2 pad 2: unconnected-(D2-A-Pad2) -> LED2
- D3 pad 1: unconnected-(D3-K-Pad1) -> GND
- D3 pad 2: unconnected-(D3-A-Pad2) -> LED3
- D4 pad 1: unconnected-(D4-K-Pad1) -> GND
- D4 pad 2: unconnected-(D4-A-Pad2) -> LED4
Routing:
- net (no net): track 0.00 -> 1.88 mm
- added copper zone on B.Cu, net GND
- added copper zone on F.Cu, net GND
Changed lines of the file:
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@@
   )
   (net 0 "")
-  (net 1 "unconnected-(D1-K-Pad1)")
-  (net 2 "unconnected-(D1-A-Pad2)")
-  (net 3 "LED2")
-  (net 4 "LED1")
-  (net 5 "LED3")
-  (net 6 "Footswitch_1")
-  (net 7 "LED4")
-  (net 8 "Footswitch_2")
-  (net 9 "GND")
-  (net 10 "Footswitch_3")
-  (net 11 "+3.3V")
-  (net 12 "Footswitch_4")
-  (net 13 "unconnected-(D2-K-Pad1)")
-  (net 14 "unconnected-(D2-A-Pad2)")
-  (net 15 "unconnected-(D3-K-Pad1)")
-  (net 16 "unconnected-(D3-A-Pad2)")
-  (net 17 "unconnected-(D4-K-Pad1)")
-  (net 18 "unconnected-(D4-A-Pad2)")
+  (net 1 "LED2")
+  (net 2 "LED1")
+  (net 3 "LED3")
+  (net 4 "Footswitch_1")
+  (net 5 "LED4")
+  (net 6 "Footswitch_2")
+  (net 7 "GND")
+  (net 8 "Footswitch_3")
+  (net 9 "+3.3V")
+  (net 10 "Footswitch_4")
   (footprint "LED_THT:LED_D5.0mm" (layer "F.Cu")
     (at 43.056 88.992)
@@
       (stroke (width 0.1) (type solid)) (fill none) (layer "F.Fab"))
     (pad "1" thru_hole rect (at 0 0) (size 1.8 1.8) (drill 0.9) (layers "*.Cu" "*.Mask")
-      (net 1 "unconnected-(D1-K-Pad1)") (pinfunction "K") (pintype "passive"))
+      (net 7 "GND") (pinfunction "K") (pintype "passive"))
     (pad "2" thru_hole circle (at 2.54 0) (size 1.8 1.8) (drill 0.9) (layers "*.Cu" "*.Mask")
-      (net 2 "unconnected-(D1-A-Pad2)") (pinfunction "A") (pintype "passive"))
+      (net 2 "LED1") (pinfunction "A") (pintype "passive"))
     (model "${KICAD6_3DMODEL_DIR}/LED_THT.3dshapes/LED_D5.0mm.wrl"
       (offset (xyz 0 0 0))
@@
       (stroke (width 0.1) (type solid)) (fill none) (layer "F.Fab"))
     (pad "1" thru_hole rect (at 0 0) (size 1.8 1.8) (drill 0.9) (layers "*.Cu" "*.Mask")
-      (net 13 "unconnected-(D2-K-Pad1)") (pinfunction "K") (pintype "passive"))
+      (net 7 "GND") (pinfunction "K") (pintype "passive"))
     (pad "2" thru_hole circle (at 2.54 0) (size 1.8 1.8) (drill 0.9) (layers "*.Cu" "*.Mask")
-      (net 14 "unconnected-(D2-A-Pad2)") (pinfunction "A") (pintype "passive"))
+      (net 1 "LED2") (pinfunction "A") (pintype "passive"))
     (model "${KICAD6_3DMODEL_DIR}/LED_THT.3dshapes/LED_D5.0mm.wrl"
       (offset (xyz 0 0 0))
@@
       (stroke (width 0.1) (type solid)) (fill none) (layer "F.Fab"))
     (pad "1" thru_hole rect (at 0 0) (size 1.8 1.8) (drill 0.9) (layers "*.Cu" "*.Mask")
-      (net 15 "unconnected-(D3-K-Pad1)") (pinfunction "K") (pintype "passive"))
+      (net 7 "GND") (pinfunction "K") (pintype "passive"))
     (pad "2" thru_hole circle (at 2.54 0) (size 1.8 1.8) (drill 0.9) (layers "*.Cu" "*.Mask")
-      (net 16 "unconnected-(D3-A-Pad2)") (pinfunction "A") (pintype "passive"))
+      (net 3 "LED3") (pinfunction "A") (pintype "passive"))
     (model "${KICAD6_3DMODEL_DIR}/LED_THT.3dshapes/LED_D5.0mm.wrl"
       (offset (xyz 0 0 0))
@@
       (stroke (width 0.1) (type solid)) (layer "F.Fab"))
     (pad "1" thru_hole roundrect (at 0 0 270) (size 1.7 1.7) (drill 1) (layers "*.Cu" "*.Mask") (roundrect_rratio 0.147059)
-      (net 3 "LED2") (pinfunction "Pin_1") (pintype "passive"))
+      (net 1 "LED2") (pinfunction "Pin_1") (pintype "passive"))
     (pad "2" thru_hole circle (at 2.54 0 270) (size 1.7 1.7) (drill 1) (layers "*.Cu" "*.Mask")
-      (net 4 "LED1") (pinfunction "Pin_2") (pintype "passive"))
+      (net 2 "LED1") (pinfunction "Pin_2") (pintype "passive"))
     (pad "3" thru_hole circle (at 0 2.54 270) (size 1.7 1.7) (drill 1) (layers "*.Cu" "*.Mask")
-      (net 5 "LED3") (pinfunction "Pin_3") (pintype "passive"))
+      (net 3 "LED3") (pinfunction "Pin_3") (pintype "passive"))
     (pad "4" thru_hole circle (at 2.54 2.54 270) (size 1.7 1.7) (drill 1) (layers "*.Cu" "*.Mask")
-      (net 6 "Footswitch_1") (pinfunction "Pin_4") (pintype "passive"))
+      (net 4 "Footswitch_1") (pinfunction "Pin_4") (pintype "passive"))
     (pad "5" thru_hole circle (at 0 5.08 270) (size 1.7 1.7) (drill 1) (layers "*.Cu" "*.Mask")
-      (net 7 "LED4") (pinfunction "Pin_5") (pintype "passive"))
+      (net 5 "LED4") (pinfunction "Pin_5") (pintype "passive"))
     (pad "6" thru_hole circle (at 2.54 5.08 270) (size 1.7 1.7) (drill 1) (layers "*.Cu" "*.Mask")
-      (net 8 "Footswitch_2") (pinfunction "Pin_6") (pintype "passive"))
+      (net 6 "Footswitch_2") (pinfunction "Pin_6") (pintype "passive"))
     (pad "7" thru_hole circle (at 0 7.62 270) (size 1.7 1.7) (drill 1) (layers "*.Cu" "*.Mask")
-      (net 9 "GND") (pinfunction "Pin_7") (pintype "passive"))
+      (net 7 "GND") (pinfunction "Pin_7") (pintype "passive"))
     (pad "8" thru_hole circle (at 2.54 7.62 270) (size 1.7 1.7) (drill 1) (layers "*.Cu" "*.Mask")
-      (net 10 "Footswitch_3") (pinfunction "Pin_8") (pintype "passive"))
+      (net 8 "Footswitch_3") (pinfunction "Pin_8") (pintype "passive"))
     (pad "9" thru_hole circle (at 0 10.16 270) (size 1.7 1.7) (drill 1) (layers "*.Cu" "*.Mask")
-      (net 11 "+3.3V") (pinfunction "Pin_9") (pintype "passive"))
+      (net 9 "+3.3V") (pinfunction "Pin_9") (pintype "passive"))
     (pad "10" thru_hole circle (at 2.54 10.16 270) (size 1.7 1.7) (drill 1) (layers "*.Cu" "*.Mask")
-      (net 12 "Footswitch_4") (pinfunction "Pin_10") (pintype "passive"))
+      (net 10 "Footswitch_4") (pinfunction "Pin_10") (pintype "passive"))
     (model "${KICAD6_3DMODEL_DIR}/Connector_IDC.3dshapes/IDC-Header_2x05_P2.54mm_Vertical.wrl"
       (offset (xyz 0 0 0))
@@
       (stroke (width 0.1) (type solid)) (fill none) (layer "F.Fab"))
     (pad "1" thru_hole rect (at 0 0) (size 1.8 1.8) (drill 0.9) (layers "*.Cu" "*.Mask")
-      (net 17 "unconnected-(D4-K-Pad1)") (pinfunction "K") (pintype "passive"))
+      (net 7 "GND") (pinfunction "K") (pintype "passive"))
     (pad "2" thru_hole circle (at 2.54 0) (size 1.8 1.8) (drill 0.9) (layers "*.Cu" "*.Mask")
-      (net 18 "unconnected-(D4-A-Pad2)") (pinfunction "A") (pintype "passive"))
+      (net 5 "LED4") (pinfunction "A") (pintype "passive"))
     (model "${KICAD6_3DMODEL_DIR}/LED_THT.3dshapes/LED_D5.0mm.wrl"
       (offset (xyz 0 0 0))
@@
   (gr_rect (start 15.202 84.29) (end 280.202 114.29)
     (stroke (width 0.2) (type default)) (fill none) (layer "F.Cu"))
+  (segment (start 172.552 99.54) (end 173.482 98.61) (width 0.25) (layer "F.Cu") (net 0))
+  (segment (start 173.482 98.61) (end 173.482 98.044) (width 0.25) (layer "F.Cu") (net 0))
+  (zone (net 7) (net_name "GND") (layers "F&B.Cu") (hatch edge 0.5)
+    (connect_pads yes (clearance 0.5))
+    (min_thickness 0.25) (filled_areas_thickness no)
+    (fill yes (thermal_gap 0.5) (thermal_bridge_width 0.5))
+    (polygon
+      (pts
+        (xy 15.202 84.29)
+        (xy 280.202 84.29)
+        (xy 280.202 114.29)
+        (xy 15.202 114.29)
+      )
+    )
+  )
   (group "" (id 2efd092d-d7d6-46f1-9215-4089ada2fd88)
     (members

Commit message: updated symbol for 3pdt, created connections
Connections:
- SW1 pad 1: (no net) -> unconnected-(SW1-Pad1)
- SW1 pad 2: (no net) -> unconnected-(SW1-Pad2)
- SW1 pad 3: (no net) -> unconnected-(SW1-Pad3)
- SW1 pad 4: (no net) -> +3.3V
- SW1 pad 5: (no net) -> Footswitch_1
- SW1 pad 6: (no net) -> GND
- SW1 pad 7: (no net) -> unconnected-(SW1-Pad7)
- SW1 pad 8: (no net) -> unconnected-(SW1-Pad8)
- SW1 pad 9: (no net) -> unconnected-(SW1-Pad9)
- SW2 pad 1: (no net) -> unconnected-(SW2-Pad1)
- SW2 pad 2: (no net) -> unconnected-(SW2-Pad2)
- SW2 pad 3: (no net) -> unconnected-(SW2-Pad3)
- SW2 pad 4: (no net) -> +3.3V
- SW2 pad 5: (no net) -> Footswitch_2
- SW2 pad 6: (no net) -> GND
- SW2 pad 7: (no net) -> unconnected-(SW2-Pad7)
- SW2 pad 8: (no net) -> unconnected-(SW2-Pad8)
- SW2 pad 9: (no net) -> unconnected-(SW2-Pad9)
- SW3 pad 1: (no net) -> unconnected-(SW3-Pad1)
- SW3 pad 2: (no net) -> unconnected-(SW3-Pad2)
- SW3 pad 3: (no net) -> unconnected-(SW3-Pad3)
- SW3 pad 4: (no net) -> +3.3V
- SW3 pad 5: (no net) -> Footswitch_3
- SW3 pad 6: (no net) -> GND
- SW3 pad 7: (no net) -> unconnected-(SW3-Pad7)
- SW3 pad 8: (no net) -> unconnected-(SW3-Pad8)
- SW3 pad 9: (no net) -> unconnected-(SW3-Pad9)
- SW4 pad 1: (no net) -> unconnected-(SW4-Pad1)
- SW4 pad 2: (no net) -> unconnected-(SW4-Pad2)
- SW4 pad 3: (no net) -> unconnected-(SW4-Pad3)
- SW4 pad 4: (no net) -> +3.3V
- SW4 pad 5: (no net) -> Footswitch_4
- SW4 pad 6: (no net) -> GND
- SW4 pad 7: (no net) -> unconnected-(SW4-Pad7)
- SW4 pad 8: (no net) -> unconnected-(SW4-Pad8)
- SW4 pad 9: (no net) -> unconnected-(SW4-Pad9)
Routing:
- net +3.3V: track 0.00 -> 235.6 mm
- net Footswitch_1: track 0.00 -> 193.2 mm, vias 0 -> 1
- net LED1: track 0.00 -> 189.9 mm
- net Footswitch_2: track 0.00 -> 122.8 mm, vias 0 -> 1
- net LED2: track 0.00 -> 115.2 mm
- net Footswitch_3: track 0.00 -> 45.3 mm, vias 0 -> 1
- net LED3: track 0.00 -> 43.4 mm
- net Footswitch_4: track 0.00 -> 37.0 mm
- net LED4: track 0.00 -> 31.6 mm
- net unconnected-(SW3-Pad3): track 0.00 -> 1.88 mm
- net (no net): track 1.88 -> 0.00 mm
- net GND: vias 0 -> 73

Commit message: gerber added
Other:
- board text added: "SW1"
- board text added: "SW2"
- board text added: "SW3"
- board text added: "SW4"
Changed lines of the file:
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@@
       (plot_on_all_layers_selection 0x0000000_00000000)
       (disableapertmacros false)
-      (usegerberextensions false)
-      (usegerberattributes true)
-      (usegerberadvancedattributes true)
-      (creategerberjobfile true)
+      (usegerberextensions true)
+      (usegerberattributes false)
+      (usegerberadvancedattributes false)
+      (creategerberjobfile false)
       (dashed_line_dash_ratio 12.000000)
       (dashed_line_gap_ratio 3.000000)
@@
       (psa4output false)
       (plotreference true)
-      (plotvalue true)
+      (plotvalue false)
       (plotinvisibletext false)
       (sketchpadsonfab false)
-      (subtractmaskfromsilk false)
+      (subtractmaskfromsilk true)
       (outputformat 1)
       (mirror false)
-      (drillshape 1)
+      (drillshape 0)
       (scaleselection 1)
-      (outputdirectory "")
+      (outputdirectory "gerbers/")
     )
   )
@@
     (fp_line (start 5.72 15.26) (end -3.18 15.26)
       (stroke (width 0.1) (type solid)) (layer "F.Fab"))
-    (pad "1" thru_hole roundrect (at 0 0 270) (size 1.7 1.7) (drill 1) (layers "*.Cu" "*.Mask") (roundrect_rratio 0.147059)
+    (pad "1" thru_hole roundrect (at 0 0 270) (size 1.7 1.7) (drill 1) (layers "*.Cu" "*.Mask") (roundrect_rratio 0.1470588235)
       (net 1 "LED2") (pinfunction "Pin_1") (pintype "passive"))
     (pad "2" thru_hole circle (at 2.54 0 270) (size 1.7 1.7) (drill 1) (layers "*.Cu" "*.Mask")
@@
   (gr_rect (start 15.202 84.29) (end 280.202 114.29)
     (stroke (width 0.2) (type default)) (fill none) (layer "F.Cu"))
+  (gr_text "SW4" (at 228.346 105.664) (layer "F.SilkS")
+    (effects (font (size 2 2) (thickness 0.2)) (justify left bottom))
+  )
+  (gr_text "SW1" (at 28.702 105.664) (layer "F.SilkS")
+    (effects (font (size 2 2) (thickness 0.2)) (justify left bottom))
+  )
+  (gr_text "SW3" (at 161.798 105.664) (layer "F.SilkS")
+    (effects (font (size 2 2) (thickness 0.2)) (justify left bottom))
+  )
+  (gr_text "SW2" (at 95.25 105.664) (layer "F.SilkS")
+    (effects (font (size 2 2) (thickness 0.2)) (justify left bottom))
+  )
   (segment (start 222.926 88.306) (end 222.926 91.477) (width 0.508) (layer "B.Cu") (net 1))
   (segment (start 166.786 88.992) (end 168.656 87.122) (width 0.508) (layer "B.Cu") (net 1))

Commit message: footswitches are now 70mm apart
Parts:
- moved SW4 11.1 mm to (255.0, 104.3)
- moved D4 10.8 mm to (253.5, 89.3)
- moved SW3 7.60 mm to (185.0, 104.3)
- moved D3 7.31 mm to (183.5, 89.3)
- moved SW2 4.15 mm to (115.0, 104.3)
- moved D2 3.86 mm to (113.5, 89.3)
- moved SW1 0.73 mm to (45.0, 104.3)
- moved D1 0.48 mm to (43.5, 89.3)
Routing:
- net +3.3V: track 235.6 -> 249.8 mm
- net LED4: track 31.6 -> 43.6 mm
- net Footswitch_4: track 37.0 -> 48.1 mm
- net Footswitch_3: track 45.3 -> 37.8 mm
- net LED3: track 43.4 -> 36.2 mm
- net Footswitch_2: track 122.8 -> 118.8 mm
- net LED2: track 115.2 -> 111.5 mm
- net unconnected-(SW3-Pad3): track 1.88 -> 0.00 mm
- net GND: vias 73 -> 43
Other:
- board outline added: 234.7 x 30 mm
- board text added: "Author: Papp Áron Date: 2024.04.08. BME VIK Diplomaterv 1 stm_audio_board_V3_Footswitch_board Repo: https://github.com/Papproni/Digital_guitar_effect"
